Commit message: add moveit simulation

File: src/hex_arm_description/urdf/firefly_y6.ros2_control.xacro (robot description, xacro)
@@ -1,5 +1,5 @@
 <?xml version="1.0"?>
 <robot xmlns:xacro="http://www.ros.org/wiki/xacro">
-  <xacro:macro name="firefly_y6_ros2_control" params="backend state_timeout_sec:=0.100">
+  <xacro:macro name="firefly_y6_ros2_control" params="backend state_timeout_sec:=0.100 activation_timeout_sec:=5.0">
     <ros2_control name="FireflyY6System" type="system">
       <hardware>
@@ -11,4 +11,5 @@
           <param name="deactivate_service">/hex_arm_bridge/deactivate_hardware</param>
           <param name="state_timeout_sec">${state_timeout_sec}</param>
+          <param name="activation_timeout_sec">${activation_timeout_sec}</param>
           <param name="service_timeout_sec">5.0</param>
         </xacro:if>

Commit message: feat(bringup): add ordered startup and harden real-arm execution
Add supervised Meow startup and improve the ROS 2/MoveIt 2 hardware
execution path for the Firefly Y6.

- Configure controllers and verify feedback before enabling hardware.
- Align J6 when needed, then move J2, J4 and J3 in order while preserving
  measured positions on joints awaiting their turn.
- Add bounded retries for hardware status queries before activation.
- Stream position and velocity commands and fix interpolation duration
  selection for nonzero endpoint velocities.
- Isolate bridge streaming from management callbacks and improve
  activation synchronization, shutdown and executor cleanup.
- Support configurable CAN interfaces with adapter identity checks.
- Set the mock initial pose and startup_ready state to
  [0, -1.350, 3.000, -0.300, 0, 0].
- Add commissioning tools, regression tests and hardware trial records.
- Update deployment documentation with current parameters and next steps.

Validation includes 45 targeted Python tests, complete mock startup,
and can2 hardware startup, small-motion execution and holding trials.

Full-workspace validation remains pending. A J2 return-motion goal
tolerance failure remains a regression case for further tuning.

File: src/hex_arm_description/urdf/firefly_y6.ros2_control.xacro (robot description, xacro)
@@ -1,5 +1,5 @@
 <?xml version="1.0"?>
 <robot xmlns:xacro="http://www.ros.org/wiki/xacro">
-  <xacro:macro name="firefly_y6_ros2_control" params="backend state_timeout_sec:=0.100 activation_timeout_sec:=5.0">
+  <xacro:macro name="firefly_y6_ros2_control" params="backend initial_positions state_timeout_sec:=0.100 activation_timeout_sec:=5.0">
     <ros2_control name="FireflyY6System" type="system">
       <hardware>
@@ -26,5 +26,5 @@
         <command_interface name="position"><param name="min">-2.86</param><param name="max">2.86</param></command_interface>
         <command_interface name="velocity"><param name="min">-6.0</param><param name="max">6.0</param></command_interface>
-        <state_interface name="position"><param name="initial_value">0.0</param></state_interface>
+        <state_interface name="position"><param name="initial_value">${initial_positions['joint_1']}</param></state_interface>
         <state_interface name="velocity"/>
         <state_interface name="effort"/>
@@ -33,5 +33,5 @@
         <command_interface name="position"><param name="min">-1.57</param><param name="max">2.09</param></command_interface>
         <command_interface name="velocity"><param name="min">-6.0</param><param name="max">6.0</param></command_interface>
-        <state_interface name="position"><param name="initial_value">0.0</param></state_interface>
+        <state_interface name="position"><param name="initial_value">${initial_positions['joint_2']}</param></state_interface>
         <state_interface name="velocity"/>
         <state_interface name="effort"/>
@@ -40,5 +40,5 @@
         <command_interface name="position"><param name="min">0.0</param><param name="max">3.14</param></command_interface>
         <command_interface name="velocity"><param name="min">-6.0</param><param name="max">6.0</param></command_interface>
-        <state_interface name="position"><param name="initial_value">1.57</param></state_interface>
+        <state_interface name="position"><param name="initial_value">${initial_positions['joint_3']}</param></state_interface>
         <state_interface name="velocity"/>
         <state_interface name="effort"/>
@@ -47,5 +47,5 @@
         <command_interface name="position"><param name="min">-1.57</param><param name="max">1.57</param></command_interface>
         <command_interface name="velocity"><param name="min">-6.0</param><param name="max">6.0</param></command_interface>
-        <state_interface name="position"><param name="initial_value">0.0</param></state_interface>
+        <state_interface name="position"><param name="initial_value">${initial_positions['joint_4']}</param></state_interface>
         <state_interface name="velocity"/>
         <state_interface name="effort"/>
@@ -54,5 +54,5 @@
         <command_interface name="position"><param name="min">-1.54</param><param name="max">1.54</param></command_interface>
         <command_interface name="velocity"><param name="min">-6.0</param><param name="max">6.0</param></command_interface>
-        <state_interface name="position"><param name="initial_value">0.0</param></state_interface>
+        <state_interface name="position"><param name="initial_value">${initial_positions['joint_5']}</param></state_interface>
         <state_interface name="velocity"/>
         <state_interface name="effort"/>
@@ -61,5 +61,5 @@
         <command_interface name="position"><param name="min">-2.79</param><param name="max">2.79</param></command_interface>
         <command_interface name="velocity"><param name="min">-6.0</param><param name="max">6.0</param></command_interface>
-        <state_interface name="position"><param name="initial_value">0.0</param></state_interface>
+        <state_interface name="position"><param name="initial_value">${initial_positions['joint_6']}</param></state_interface>
         <state_interface name="velocity"/>
         <state_interface name="effort"/>

File: src/hex_arm_description/urdf/firefly_y6.urdf.xacro (robot description, xacro)
@@ -4,4 +4,6 @@
   <xacro:arg name="controllers_file" default=""/>
   <xacro:arg name="state_timeout_sec" default="0.100"/>
+  <xacro:arg name="initial_positions_file" default=""/>
+  <xacro:property name="initial_positions" value="${xacro.load_yaml('$(arg initial_positions_file)')['initial_positions'] if '$(arg initial_positions_file)' else dict(joint_1=0.0, joint_2=0.0, joint_3=1.57, joint_4=0.0, joint_5=0.0, joint_6=0.0)}"/>
   <!-- Geometry, inertials, joint origins, axes, and limits remain owned by the
        pinned upstream package. The contract test compares every field. -->
@@ -9,5 +11,5 @@
   <xacro:include filename="$(find hex_arm_description)/urdf/firefly_y6.ros2_control.xacro"/>
   <xacro:if value="${'$(arg backend)' != 'view'}">
-    <xacro:firefly_y6_ros2_control backend="$(arg backend)" state_timeout_sec="$(arg state_timeout_sec)"/>
+    <xacro:firefly_y6_ros2_control backend="$(arg backend)" state_timeout_sec="$(arg state_timeout_sec)" initial_positions="${initial_positions}"/>
   </xacro:if>
   <xacro:if value="${'$(arg backend)' == 'gz'}">

Commit message: feat: streamline real-arm runtime and add damped shutdown
Refactor the Firefly Y6 control stack for a smaller production runtime,
consistent joint coordinates, and guarded real-hardware shutdown.

- Split the Rust controller into reusable motor backends, runtime services,
  startup recipes, and opt-in commissioning tools.
- Make the controller robot_api.proto the single protocol authority and
  generate the Python bridge bindings from it.
- Move J3 to the corrected coordinate system where the former 1.57 rad
  position is zero, and update URDF, SRDF, limits, startup poses, MoveIt
  configuration, profiles, and tests consistently.
- Define the power-cycle folded pose as
  [0, -1.570, 1.570, 0, 0, 0] and startup_ready as
  [0, -1.350, 1.430, -0.300, 0, 0].
- Preserve the mandatory J2 -> J4 -> J3 startup sequence through a shared
  startup recipe.
- Isolate view-launch joint-state and TF namespaces to prevent duplicate
  publishers and jumping models.
- Add a guarded normal-exit workflow that cancels active motion, returns to
  startup_ready through strict MoveIt planning, verifies stationary feedback,
  and transfers terminal control to the Rust driver.
- Ramp position stiffness and gravity feed-forward to zero while applying
  configurable velocity damping, then require unloaded settling near the
  folded pose before confirmed all-axis disable.
- Keep faults, incomplete startup, SIGTERM, repeated Ctrl-C, stale feedback,
  overspeed, timeout, and planning failure on the immediate fail-closed
  shutdown path.
- Preserve structured disable acknowledgements independently from the
  soft-stop result and retry unconfirmed disable without reopening commands.
- Add a self-contained production Docker image and Compose deployment with
  scoped signal forwarding and a 180-second shutdown grace period.
- Expand Rust, bridge, bringup, signal-ordering, profile, MoveIt, and shutdown
  regression coverage and update the bilingual operation documentation.

File: src/hex_arm_description/urdf/firefly_y6.ros2_control.xacro (robot description, xacro)
@@ -38,5 +38,5 @@
       </joint>
       <joint name="joint_3">
-        <command_interface name="position"><param name="min">0.0</param><param name="max">3.14</param></command_interface>
+        <command_interface name="position"><param name="min">-1.57</param><param name="max">1.57</param></command_interface>
         <command_interface name="velocity"><param name="min">-6.0</param><param name="max">6.0</param></command_interface>
         <state_interface name="position"><param name="initial_value">${initial_positions['joint_3']}</param></state_interface>

File: src/hex_arm_description/urdf/firefly_y6.urdf.xacro (robot description, xacro)
@@ -5,5 +5,5 @@
   <xacro:arg name="state_timeout_sec" default="0.100"/>
   <xacro:arg name="initial_positions_file" default=""/>
-  <xacro:property name="initial_positions" value="${xacro.load_yaml('$(arg initial_positions_file)')['initial_positions'] if '$(arg initial_positions_file)' else dict(joint_1=0.0, joint_2=0.0, joint_3=1.57, joint_4=0.0, joint_5=0.0, joint_6=0.0)}"/>
+  <xacro:property name="initial_positions" value="${xacro.load_yaml('$(arg initial_positions_file)')['initial_positions'] if '$(arg initial_positions_file)' else dict(joint_1=0.0, joint_2=0.0, joint_3=0.0, joint_4=0.0, joint_5=0.0, joint_6=0.0)}"/>
   <!-- Geometry, inertials, joint origins, axes, and limits remain owned by the
        pinned upstream package. The contract test compares every field. -->

File: src/xpkg_urdf_firefly_y6/urdf/xpkg_urdf_firefly_y6.urdf (robot description, URDF)
Before this commit: robot firefly_y6, 7 links, 6 joints
Joints:
- joint joint_3: limit lower=0 upper=3.14 effort=6 velocity=6 -> lower=-1.57 upper=1.57 effort=6 velocity=6; origin xyz=0 0 0.27 rpy=0 0 0 -> xyz=0 0 0.27 rpy=0 1.57 0

Commit message: feat: replace Python bridge with direct C++ Zenoh
 - Route real arm control directly from the C++ ros2_control plugin to the
Rust driver over Zenoh. Use bounded atomic snapshot mailboxes for realtime
read/write, enforce command sequence, activation generation, and age, and
deliver feedback directly to the hardware interface.

File: src/hex_arm_description/urdf/firefly_y6.ros2_control.xacro (robot description, xacro)
@@ -1,16 +1,17 @@
 <?xml version="1.0"?>
 <robot xmlns:xacro="http://www.ros.org/wiki/xacro">
-  <xacro:macro name="firefly_y6_ros2_control" params="backend initial_positions state_timeout_sec:=0.100 activation_timeout_sec:=5.0">
+  <xacro:macro name="firefly_y6_ros2_control" params="backend initial_positions state_timeout_sec:=0.100 activation_timeout_sec:=5.0 zenoh_connect:='tcp/127.0.0.1:7448' robot_prefix:='hexmeow/ubuntu/firefly_y6_meow' command_period_sec:=0.01 startup_timeout_sec:=30.0">
     <ros2_control name="FireflyY6System" type="system">
       <hardware>
         <xacro:if value="${backend == 'real'}">
           <plugin>hex_arm_hardware/HexArmSystem</plugin>
-          <param name="command_topic">/hex_arm/internal/command</param>
-          <param name="state_topic">/hex_arm/internal/state</param>
-          <param name="activate_service">/hex_arm_bridge/activate_hardware</param>
-          <param name="deactivate_service">/hex_arm_bridge/deactivate_hardware</param>
+          <param name="zenoh_connect">${zenoh_connect}</param>
+          <param name="robot_prefix">${robot_prefix}</param>
+          <param name="command_period_sec">${command_period_sec}</param>
+          <param name="startup_timeout_sec">${startup_timeout_sec}</param>
+          <param name="command_max_age_sec">0.05</param>
           <param name="state_timeout_sec">${state_timeout_sec}</param>
           <param name="activation_timeout_sec">${activation_timeout_sec}</param>
-          <!-- Must exceed the bridge's 5 s serialized six-axis transition timeout. -->
+          <!-- Must exceed the driver's 5 s serialized six-axis transition timeout. -->
           <param name="service_timeout_sec">10.0</param>
         </xacro:if>

File: src/hex_arm_description/urdf/firefly_y6.urdf.xacro (robot description, xacro)
@@ -5,4 +5,8 @@
   <xacro:arg name="state_timeout_sec" default="0.100"/>
   <xacro:arg name="initial_positions_file" default=""/>
+  <xacro:arg name="zenoh_connect" default="tcp/127.0.0.1:7448"/>
+  <xacro:arg name="robot_prefix" default="hexmeow/ubuntu/firefly_y6_meow"/>
+  <xacro:arg name="command_period_sec" default="0.01"/>
+  <xacro:arg name="startup_timeout_sec" default="30.0"/>
   <xacro:property name="initial_positions" value="${xacro.load_yaml('$(arg initial_positions_file)')['initial_positions'] if '$(arg initial_positions_file)' else dict(joint_1=0.0, joint_2=0.0, joint_3=0.0, joint_4=0.0, joint_5=0.0, joint_6=0.0)}"/>
   <!-- Geometry, inertials, joint origins, axes, and limits remain owned by the
@@ -11,5 +15,8 @@
   <xacro:include filename="$(find hex_arm_description)/urdf/firefly_y6.ros2_control.xacro"/>
   <xacro:if value="${'$(arg backend)' != 'view'}">
-    <xacro:firefly_y6_ros2_control backend="$(arg backend)" state_timeout_sec="$(arg state_timeout_sec)" initial_positions="${initial_positions}"/>
+    <xacro:firefly_y6_ros2_control backend="$(arg backend)" state_timeout_sec="$(arg state_timeout_sec)" initial_positions="${initial_positions}"
+      zenoh_connect="$(arg zenoh_connect)"
+      robot_prefix="$(arg robot_prefix)" command_period_sec="$(arg command_period_sec)"
+      startup_timeout_sec="$(arg startup_timeout_sec)"/>
   </xacro:if>
   <xacro:if value="${'$(arg backend)' == 'gz'}">

Commit message: feat: make the arm stack composable and restore verified startup
- Add per-instance namespaces and joint prefixes, composable robot
  descriptions, shared controller support, and multi-arm integration examples.
- Extract the shared protocol and bringup utilities into installable packages;
  make hardware and controller builds portable across workspaces.
- Separate optional simulation and visualization dependencies from core bringup.
- Add stop-operation ownership, verified disable receipts, and trajectory
  timing and interpolation diagnostics.
- Set the shutdown path tolerance to 0.11 rad and update deployment guidance
  and integration coverage.

File: src/hex_arm_description/urdf/firefly_y6.ros2_control.xacro (robot description, xacro)
@@ -1,6 +1,6 @@
 <?xml version="1.0"?>
 <robot xmlns:xacro="http://www.ros.org/wiki/xacro">
-  <xacro:macro name="firefly_y6_ros2_control" params="backend initial_positions state_timeout_sec:=0.100 activation_timeout_sec:=5.0 zenoh_connect:='tcp/127.0.0.1:7448' robot_prefix:='hexmeow/ubuntu/firefly_y6_meow' command_period_sec:=0.01 startup_timeout_sec:=30.0">
-    <ros2_control name="FireflyY6System" type="system">
+  <xacro:macro name="firefly_y6_ros2_control" params="backend initial_positions state_timeout_sec:=0.100 activation_timeout_sec:=5.0 zenoh_connect:='tcp/127.0.0.1:7448' robot_prefix:='hexmeow/ubuntu/firefly_y6_meow' command_period_sec:=0.01 startup_timeout_sec:=30.0 prefix:='' hardware_name:='FireflyY6System' ros_namespace:=''">
+    <ros2_control name="${hardware_name}" type="system">
       <hardware>
         <xacro:if value="${backend == 'real'}">
@@ -8,4 +8,5 @@
           <param name="zenoh_connect">${zenoh_connect}</param>
           <param name="robot_prefix">${robot_prefix}</param>
+          <param name="ros_namespace">${ros_namespace}</param>
           <param name="command_period_sec">${command_period_sec}</param>
           <param name="startup_timeout_sec">${startup_timeout_sec}</param>
@@ -24,5 +25,6 @@
         </xacro:if>
       </hardware>
-      <joint name="joint_1">
+      <joint name="${prefix}joint_1">
+        <param name="device_joint_name">joint_1</param>
         <command_interface name="position"><param name="min">-2.86</param><param name="max">2.86</param></command_interface>
         <command_interface name="velocity"><param name="min">-6.0</param><param name="max">6.0</param></command_interface>
@@ -31,5 +33,6 @@
         <state_interface name="effort"/>
       </joint>
-      <joint name="joint_2">
+      <joint name="${prefix}joint_2">
+        <param name="device_joint_name">joint_2</param>
         <command_interface name="position"><param name="min">-1.57</param><param name="max">2.09</param></command_interface>
         <command_interface name="velocity"><param name="min">-6.0</param><param name="max">6.0</param></command_interface>
@@ -38,5 +41,6 @@
         <state_interface name="effort"/>
       </joint>
-      <joint name="joint_3">
+      <joint name="${prefix}joint_3">
+        <param name="device_joint_name">joint_3</param>
         <command_interface name="position"><param name="min">-1.57</param><param name="max">1.57</param></command_interface>
         <command_interface name="velocity"><param name="min">-6.0</param><param name="max">6.0</param></command_interface>
@@ -45,5 +49,6 @@
         <state_interface name="effort"/>
       </joint>
-      <joint name="joint_4">
+      <joint name="${prefix}joint_4">
+        <param name="device_joint_name">joint_4</param>
         <command_interface name="position"><param name="min">-1.57</param><param name="max">1.57</param></command_interface>
         <command_interface name="velocity"><param name="min">-6.0</param><param name="max">6.0</param></command_interface>
@@ -52,5 +57,6 @@
         <state_interface name="effort"/>
       </joint>
-      <joint name="joint_5">
+      <joint name="${prefix}joint_5">
+        <param name="device_joint_name">joint_5</param>
         <command_interface name="position"><param name="min">-1.54</param><param name="max">1.54</param></command_interface>
         <command_interface name="velocity"><param name="min">-6.0</param><param name="max">6.0</param></command_interface>
@@ -59,5 +65,6 @@
         <state_interface name="effort"/>
       </joint>
-      <joint name="joint_6">
+      <joint name="${prefix}joint_6">
+        <param name="device_joint_name">joint_6</param>
         <command_interface name="position"><param name="min">-2.79</param><param name="max">2.79</param></command_interface>
         <command_interface name="velocity"><param name="min">-6.0</param><param name="max">6.0</param></command_interface>

File: src/hex_arm_description/urdf/firefly_y6.urdf.xacro (robot description, xacro)
@@ -9,20 +9,29 @@
   <xacro:arg name="command_period_sec" default="0.01"/>
   <xacro:arg name="startup_timeout_sec" default="30.0"/>
+  <xacro:arg name="prefix" default=""/>
+  <xacro:arg name="parent" default=""/>
+  <xacro:arg name="xyz" default="0 0 0"/>
+  <xacro:arg name="rpy" default="0 0 0"/>
+  <xacro:arg name="hardware_name" default="FireflyY6System"/>
+  <xacro:arg name="ros_namespace" default=""/>
+  <xacro:arg name="tool_link" default=""/>
+  <xacro:arg name="tcp_xyz" default="0 0 0"/>
+  <xacro:arg name="tcp_rpy" default="0 0 0"/>
   <xacro:property name="initial_positions" value="${xacro.load_yaml('$(arg initial_positions_file)')['initial_positions'] if '$(arg initial_positions_file)' else dict(joint_1=0.0, joint_2=0.0, joint_3=0.0, joint_4=0.0, joint_5=0.0, joint_6=0.0)}"/>
   <!-- Geometry, inertials, joint origins, axes, and limits remain owned by the
        pinned upstream package. The contract test compares every field. -->
-  <xacro:include filename="$(find xpkg_urdf_firefly_y6)/urdf/xpkg_urdf_firefly_y6.urdf"/>
-  <xacro:include filename="$(find hex_arm_description)/urdf/firefly_y6.ros2_control.xacro"/>
-  <xacro:if value="${'$(arg backend)' != 'view'}">
-    <xacro:firefly_y6_ros2_control backend="$(arg backend)" state_timeout_sec="$(arg state_timeout_sec)" initial_positions="${initial_positions}"
-      zenoh_connect="$(arg zenoh_connect)"
-      robot_prefix="$(arg robot_prefix)" command_period_sec="$(arg command_period_sec)"
-      startup_timeout_sec="$(arg startup_timeout_sec)"/>
-  </xacro:if>
+  <xacro:include filename="$(find hex_arm_description)/urdf/firefly_y6.macro.xacro"/>
+  <xacro:firefly_y6_arm backend="$(arg backend)" prefix="$(arg prefix)"
+    parent="$(arg parent)" xyz="$(arg xyz)" rpy="$(arg rpy)"
+    hardware_name="$(arg hardware_name)" ros_namespace="$(arg ros_namespace)"
+    tool_link="$(arg tool_link)" tcp_xyz="$(arg tcp_xyz)" tcp_rpy="$(arg tcp_rpy)"
+    state_timeout_sec="$(arg state_timeout_sec)" initial_positions="${initial_positions}"
+    zenoh_connect="$(arg zenoh_connect)" robot_prefix="$(arg robot_prefix)"
+    command_period_sec="$(arg command_period_sec)" startup_timeout_sec="$(arg startup_timeout_sec)"/>
   <xacro:if value="${'$(arg backend)' == 'gz'}">
     <link name="world"/>
-    <joint name="world_to_base" type="fixed">
+    <joint name="$(arg prefix)world_to_base" type="fixed">
       <parent link="world"/>
-      <child link="base_link"/>
+      <child link="$(arg prefix)base_link"/>
     </joint>
     <gazebo>
